File: pcb/main_pcb/main_pcb.kicad_pcb (KiCad board)
At the start: 2 copper layers, 80 x 100 mm, 72 parts, among them J1 Conn_01x05, J10 Conn_01x06_Male, J11 Conn_01x04, J12 Screw_Terminal_01x02, J13 Conn_01x02_Male, J2 Conn_01x05, J3 Conn_01x05, J4 Conn_01x05, J5 Conn_01x05, J6 Conn_01x05, J7 Conn_01x04, J8 Conn_01x06_Male, J9 Conn_01x04, Q1 Q_PMOS_GDS, SW1 SW_SPDT, U1 LSM6DSO, U2 Teensy_4.1, U3 DRV8833, U4 LM1117-3.3, U5 TPIC74101

Commit message: changes to pcb
Parts:
- removed C1: 330uF, Capacitor_SMD:CP_Elec_10x10.5
- removed C10, C11, C2, C4: 0.1uF, Capacitor_SMD:C_0603_1608Metric_Pad1.08x0.95mm_HandSolder
- removed C13: 100uF, Capacitor_SMD:CP_Elec_8x10.5
- removed C14, C15, C5: 22uF, Capacitor_SMD:CP_Elec_8x10.5
- removed C3, C6: 470nF, Capacitor_SMD:C_0603_1608Metric_Pad1.08x0.95mm_HandSolder
- removed C7: 150nF, Capacitor_SMD:C_0603_1608Metric_Pad1.08x0.95mm_HandSolder
- removed C8, C9: 4.7nF, Capacitor_SMD:C_0603_1608Metric_Pad1.08x0.95mm_HandSolder
- removed D1, D2: LED, LED_THT:LED_D5.0mm
- removed D3: D, Diode_SMD:D_0805_2012Metric
- removed D4: D_Schottky, Diode_SMD:D_TUMD2
- removed J11, J9: Conn_01x04, Connector_JST:JST_XH_B4B-XH-A_1x04_P2.50mm_Vertical
- removed J12: Screw_Terminal_01x02, TerminalBlock:TerminalBlock_bornier-2_P5.08mm
- removed J13: Conn_01x02_Male, Connector_PinHeader_2.54mm:PinHeader_1x02_P2.54mm_Vertical
- removed L1, L2: 22uH, custom_footprints:L_SRR1050HA_Bourns
- removed Q1: Q_PMOS_GDS, Package_TO_SOT_SMD:TO-263-3_TabPin2
- removed R1, R3, R5, R8: 3.3k, Resistor_SMD:R_0603_1608Metric_Pad0.98x0.95mm_HandSolder
- removed R10: 0, Resistor_SMD:R_0603_1608Metric_Pad0.98x0.95mm_HandSolder
- removed R11, R12: 5k, Resistor_SMD:R_0603_1608Metric_Pad0.98x0.95mm_HandSolder
- removed R13: 470, Resistor_SMD:R_0603_1608Metric_Pad0.98x0.95mm_HandSolder
- removed R14, R15, R16, R17, R2, R4, R6: 2.2k, Resistor_SMD:R_0603_1608Metric_Pad0.98x0.95mm_HandSolder
- removed R7: 12k, Resistor_SMD:R_0603_1608Metric_Pad0.98x0.95mm_HandSolder
- removed R9: 4.53k, Resistor_SMD:R_0603_1608Metric_Pad0.98x0.95mm_HandSolder
- removed SW1: SW_SPDT, custom_footprints:SW_SPDT_NKK_MS12AANW03
- removed U1: LSM6DSO, custom_footprints:SENS_LSM6DSO_Pololu_2798
- removed U2: Teensy_4.1, custom_footprints:MCU_TEENSY41_PJRC
- removed U4: LM1117-3.3, Package_TO_SOT_SMD:SOT-223-3_TabPin2
- removed U5: TPIC74101, custom_footprints:HTSSOP-20-1EP_4.4x6.5mm_P0.65mm_EP3.4x6.5mm_ThermalVias
- J7: value Conn_01x04 -> Conn_01x05; footprint Connector_JST:JST_XH_B4B-XH-A_1x04_P2.50mm_Vertical -> Connector_JST:JST_XH_B5B-XH-A_1x05_P2.50mm_Vertical
- moved J7 19.9 mm to (106.8, 111.8)
Connections:
- J7 pad 1: +5V -> GND
- J7 pad 2: /microcontroller/Trig1 -> /microcontroller/SDA2
- J7 pad 3: Net-(J7-Pad3) -> /microcontroller/SCL2
- J7 pad 4: GND -> /microcontroller/LCS7
Routing:
- net (no net): track 0.00 -> 459.5 mm, vias 0 -> 9
- net /microcontroller/SCL2: track 93.5 -> 244.8 mm
- net +5V: track 94.2 -> 0.00 mm, vias 2 -> 0
- net +5VD: track 92.1 -> 0.00 mm, vias 1 -> 0
- net /microcontroller/LCS6: track 83.0 -> 0.00 mm
- net /microcontroller/LCS5: track 81.1 -> 0.00 mm
- net /microcontroller/SDA2: track 103.9 -> 184.9 mm
- net /microcontroller/LCS4: track 68.2 -> 0.00 mm
- net Net-(D1-Pad1): track 41.4 -> 0.00 mm
- net /microcontroller/Trig3: track 20.8 -> 0.00 mm
- net /microcontroller/SDA1: track 18.9 -> 0.00 mm
- net Net-(J9-Pad3): track 17.3 -> 0.00 mm
- net Net-(J11-Pad3): track 15.7 -> 0.00 mm
- net /microcontroller/Trig2: track 15.5 -> 0.00 mm
- net Net-(J7-Pad3): track 13.9 -> 0.00 mm
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- added copper zone on F.Cu, net (none)
- removed copper zone on F.Cu, net Net-(C1-Pad1)
- removed copper zone on F.Cu, net Net-(C8-Pad1)
- removed copper zone on F.Cu, net Net-(C9-Pad1)
- removed copper zone on F.Cu, net Net-(D1-Pad1)

Commit message: Error corrections
Routing:
- net /microcontroller/SCL2: track 244.8 -> 93.5 mm
- net /microcontroller/LCS6: track 0.00 -> 151.2 mm
- net /microcontroller/LCS5: track 0.00 -> 81.1 mm
- net /microcontroller/SDA2: track 184.9 -> 103.9 mm
Changed lines of the file:
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@@
       (layerselection 0x00010fc_ffffffff)
       (disableapertmacros false)
-      (usegerberextensions true)
+      (usegerberextensions false)
       (usegerberattributes true)
       (usegerberadvancedattributes true)
@@
   (segment (start 110.5 72.475) (end 110.5 59.4) (width 0.254) (layer "F.Cu") (net 22))
   (segment (start 110.5 77.5) (end 110.5 72.475) (width 0.254) (layer "F.Cu") (net 22))
-  (segment (start 93.5 64.525) (end 92.2 65.825) (width 0.25) (layer "F.Cu") (net 22))
   (segment (start 115.8875 59.5) (end 113.8 59.5) (width 0.254) (layer "F.Cu") (net 22))
-  (segment (start 110 119.7) (end 117.19 126.89) (width 0.25) (layer "F.Cu") (net 22))
   (segment (start 121 110) (end 120.5 110.5) (width 0.254) (layer "F.Cu") (net 22))
-  (segment (start 94.5 78.2) (end 105.4 78.2) (width 0.25) (layer "F.Cu") (net 22))
   (segment (start 113 106.35) (end 113 80) (width 0.254) (layer "F.Cu") (net 22))
   (segment (start 118.62 106.57) (end 120.57 106.57) (width 0.254) (layer "F.Cu") (net 22))
   (segment (start 98.5 57.5) (end 110.4 57.5) (width 0.25) (layer "F.Cu") (net 22))
-  (segment (start 105.4 78.2) (end 110 82.8) (width 0.25) (layer "F.Cu") (net 22))
   (segment (start 98.5 57.5) (end 98.5 73.525) (width 0.25) (layer "F.Cu") (net 22))
   (segment (start 117.15 110.5) (end 113 106.35) (width 0.254) (layer "F.Cu") (net 22))
@@
   (segment (start 110.5 57.4) (end 110.5 54.475) (width 0.254) (layer "F.Cu") (net 22))
   (segment (start 120.57 106.57) (end 121 107) (width 0.254) (layer "F.Cu") (net 22))
-  (segment (start 92.2 65.825) (end 92.2 75.9) (width 0.25) (layer "F.Cu") (net 22))
   (segment (start 121 107) (end 121 110) (width 0.254) (layer "F.Cu") (net 22))
   (segment (start 110.5 59.4) (end 110.5 57.4) (width 0.254) (layer "F.Cu") (net 22))
-  (segment (start 92.2 75.9) (end 94.5 78.2) (width 0.25) (layer "F.Cu") (net 22))
-  (segment (start 110 82.8) (end 110 119.7) (width 0.25) (layer "F.Cu") (net 22))
-  (segment (start 117.19 126.89) (end 118.62 126.89) (width 0.25) (layer "F.Cu") (net 22))
   (segment (start 113 80) (end 110.5 77.5) (width 0.254) (layer "F.Cu") (net 22))
   (via (at 112.2 59.5) (size 0.8) (drill 0.4) (layers "F.Cu" "B.Cu") (net 22))
@@
   (segment (start 113.8 59.5) (end 112.2 59.5) (width 0.254) (layer "B.Cu") (net 22))
   (segment (start 113 72.475) (end 113 78) (width 0.25) (layer "F.Cu") (net 23))
-  (segment (start 105.8 77.5) (end 95.3 77.5) (width 0.25) (layer "F.Cu") (net 23))
-  (segment (start 111 118.2) (end 111 82.7) (width 0.25) (layer "F.Cu") (net 23))
-  (segment (start 94.8 74.7) (end 96.9 76.8) (width 0.25) (layer "F.Cu") (net 23))
-  (segment (start 117.11 121.81) (end 118.62 121.81) (width 0.25) (layer "F.Cu") (net 23))
   (segment (start 113 78) (end 114 79) (width 0.25) (layer "F.Cu") (net 23))
   (segment (start 98.425 53.1) (end 111.625 53.1) (width 0.25) (layer "F.Cu") (net 23))
-  (segment (start 93.5 55.525) (end 94.8 56.825) (width 0.25) (layer "F.Cu") (net 23))
-  (segment (start 118.62 124.35) (end 117.15 124.35) (width 0.25) (layer "F.Cu") (net 23))
   (segment (start 96 55.525) (end 98.425 53.1) (width 0.25) (layer "F.Cu") (net 23))
-  (segment (start 96.9 76.8) (end 106.15 76.8) (width 0.25) (layer "F.Cu") (net 23))
-  (segment (start 93.5 75.7) (end 93.5 73.525) (width 0.25) (layer "F.Cu") (net 23))
   (segment (start 114 79) (end 114 104.49) (width 0.25) (layer "F.Cu") (net 23))
-  (segment (start 111 82.7) (end 105.8 77.5) (width 0.25) (layer "F.Cu") (net 23))
   (segment (start 96 73.525) (end 96 55.525) (width 0.25) (layer "F.Cu") (net 23))
-  (segment (start 94.8 56.825) (end 94.8 74.7) (width 0.25) (layer "F.Cu") (net 23))
-  (segment (start 95.3 77.5) (end 93.5 75.7) (width 0.25) (layer "F.Cu") (net 23))
-  (segment (start 112 82.65) (end 112 116.7) (width 0.25) (layer "F.Cu") (net 23))
-  (segment (start 117.15 124.35) (end 111 118.2) (width 0.25) (layer "F.Cu") (net 23))
   (segment (start 113 54.475) (end 113 72.475) (width 0.254) (layer "F.Cu") (net 23))
-  (segment (start 106.15 76.8) (end 112 82.65) (width 0.25) (layer "F.Cu") (net 23))
   (segment (start 111.625 53.1) (end 113 54.475) (width 0.25) (layer "F.Cu") (net 23))
   (segment (start 114 104.49) (end 118.62 109.11) (width 0.25) (layer "F.Cu") (net 23))
-  (segment (start 112 116.7) (end 117.11 121.81) (width 0.25) (layer "F.Cu") (net 23))
   (segment (start 126.25 133.5) (end 126.25 137.6625) (width 0.254) (layer "F.Cu") (net 24))
   (segment (start 118.62 131.97) (end 122.18 131.97) (width 0.254) (layer "F.Cu") (net 25))
@@
   (segment (start 118.62 101.49) (end 116 98.87) (width 0.254) (layer "F.Cu") (net 33))
   (segment (start 116 98.87) (end 116 75.5) (width 0.254) (layer "F.Cu") (net 33))
+  (segment (start 93.5 64.525) (end 92.2 65.825) (width 0.25) (layer "F.Cu") (net 35))
+  (segment (start 110 119.7) (end 117.19 126.89) (width 0.25) (layer "F.Cu") (net 35))
+  (segment (start 94.5 78.2) (end 105.4 78.2) (width 0.25) (layer "F.Cu") (net 35))
+  (segment (start 105.4 78.2) (end 110 82.8) (width 0.25) (layer "F.Cu") (net 35))
+  (segment (start 92.2 65.825) (end 92.2 75.9) (width 0.25) (layer "F.Cu") (net 35))
+  (segment (start 92.2 75.9) (end 94.5 78.2) (width 0.25) (layer "F.Cu") (net 35))
+  (segment (start 110 82.8) (end 110 119.7) (width 0.25) (layer "F.Cu") (net 35))
+  (segment (start 117.19 126.89) (end 118.62 126.89) (width 0.25) (layer "F.Cu") (net 35))
+  (segment (start 105.8 77.5) (end 95.3 77.5) (width 0.25) (layer "F.Cu") (net 36))
+  (segment (start 111 118.2) (end 111 82.7) (width 0.25) (layer "F.Cu") (net 36))
+  (segment (start 94.8 74.7) (end 96.9 76.8) (width 0.25) (layer "F.Cu") (net 36))
+  (segment (start 117.11 121.81) (end 118.62 121.81) (width 0.25) (layer "F.Cu") (net 36))
+  (segment (start 93.5 55.525) (end 94.8 56.825) (width 0.25) (layer "F.Cu") (net 36))
+  (segment (start 118.62 124.35) (end 117.15 124.35) (width 0.25) (layer "F.Cu") (net 36))
+  (segment (start 96.9 76.8) (end 106.15 76.8) (width 0.25) (layer "F.Cu") (net 36))
+  (segment (start 93.5 75.7) (end 93.5 73.525) (width 0.25) (layer "F.Cu") (net 36))
+  (segment (start 111 82.7) (end 105.8 77.5) (width 0.25) (layer "F.Cu") (net 36))
+  (segment (start 94.8 56.825) (end 94.8 74.7) (width 0.25) (layer "F.Cu") (net 36))
+  (segment (start 95.3 77.5) (end 93.5 75.7) (width 0.25) (layer "F.Cu") (net 36))
+  (segment (start 112 82.65) (end 112 116.7) (width 0.25) (layer "F.Cu") (net 36))
+  (segment (start 117.15 124.35) (end 111 118.2) (width 0.25) (layer "F.Cu") (net 36))
+  (segment (start 106.15 76.8) (end 112 82.65) (width 0.25) (layer "F.Cu") (net 36))
+  (segment (start 112 116.7) (end 117.11 121.81) (width 0.25) (layer "F.Cu") (net 36))
   (zone locked (net 2) (net_name "GND") (layers F&B.Cu) (hatch edge 0.508)
     (connect_pads thru_hole_only (clearance 0.254))

Commit message: changes to PCB
Routing:
- net /microcontroller/SCL2: track 93.5 -> 244.8 mm
- net /microcontroller/LCS6: track 151.2 -> 0.00 mm
- net /microcontroller/LCS5: track 81.1 -> 0.00 mm
- net /microcontroller/SDA2: track 103.9 -> 184.9 mm
Changed lines of the file:
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@@
   (segment (start 110.5 72.475) (end 110.5 59.4) (width 0.254) (layer "F.Cu") (net 22))
   (segment (start 110.5 77.5) (end 110.5 72.475) (width 0.254) (layer "F.Cu") (net 22))
+  (segment (start 93.5 64.525) (end 92.2 65.825) (width 0.25) (layer "F.Cu") (net 22))
   (segment (start 115.8875 59.5) (end 113.8 59.5) (width 0.254) (layer "F.Cu") (net 22))
+  (segment (start 110 119.7) (end 117.19 126.89) (width 0.25) (layer "F.Cu") (net 22))
   (segment (start 121 110) (end 120.5 110.5) (width 0.254) (layer "F.Cu") (net 22))
+  (segment (start 94.5 78.2) (end 105.4 78.2) (width 0.25) (layer "F.Cu") (net 22))
   (segment (start 113 106.35) (end 113 80) (width 0.254) (layer "F.Cu") (net 22))
   (segment (start 118.62 106.57) (end 120.57 106.57) (width 0.254) (layer "F.Cu") (net 22))
   (segment (start 98.5 57.5) (end 110.4 57.5) (width 0.25) (layer "F.Cu") (net 22))
+  (segment (start 105.4 78.2) (end 110 82.8) (width 0.25) (layer "F.Cu") (net 22))
   (segment (start 98.5 57.5) (end 98.5 73.525) (width 0.25) (layer "F.Cu") (net 22))
   (segment (start 117.15 110.5) (end 113 106.35) (width 0.254) (layer "F.Cu") (net 22))
@@
   (segment (start 110.5 57.4) (end 110.5 54.475) (width 0.254) (layer "F.Cu") (net 22))
   (segment (start 120.57 106.57) (end 121 107) (width 0.254) (layer "F.Cu") (net 22))
+  (segment (start 92.2 65.825) (end 92.2 75.9) (width 0.25) (layer "F.Cu") (net 22))
   (segment (start 121 107) (end 121 110) (width 0.254) (layer "F.Cu") (net 22))
   (segment (start 110.5 59.4) (end 110.5 57.4) (width 0.254) (layer "F.Cu") (net 22))
+  (segment (start 92.2 75.9) (end 94.5 78.2) (width 0.25) (layer "F.Cu") (net 22))
+  (segment (start 110 82.8) (end 110 119.7) (width 0.25) (layer "F.Cu") (net 22))
+  (segment (start 117.19 126.89) (end 118.62 126.89) (width 0.25) (layer "F.Cu") (net 22))
   (segment (start 113 80) (end 110.5 77.5) (width 0.254) (layer "F.Cu") (net 22))
   (via (at 112.2 59.5) (size 0.8) (drill 0.4) (layers "F.Cu" "B.Cu") (net 22))
@@
   (segment (start 113.8 59.5) (end 112.2 59.5) (width 0.254) (layer "B.Cu") (net 22))
   (segment (start 113 72.475) (end 113 78) (width 0.25) (layer "F.Cu") (net 23))
+  (segment (start 105.8 77.5) (end 95.3 77.5) (width 0.25) (layer "F.Cu") (net 23))
+  (segment (start 111 118.2) (end 111 82.7) (width 0.25) (layer "F.Cu") (net 23))
+  (segment (start 94.8 74.7) (end 96.9 76.8) (width 0.25) (layer "F.Cu") (net 23))
+  (segment (start 117.11 121.81) (end 118.62 121.81) (width 0.25) (layer "F.Cu") (net 23))
   (segment (start 113 78) (end 114 79) (width 0.25) (layer "F.Cu") (net 23))
   (segment (start 98.425 53.1) (end 111.625 53.1) (width 0.25) (layer "F.Cu") (net 23))
+  (segment (start 93.5 55.525) (end 94.8 56.825) (width 0.25) (layer "F.Cu") (net 23))
+  (segment (start 118.62 124.35) (end 117.15 124.35) (width 0.25) (layer "F.Cu") (net 23))
   (segment (start 96 55.525) (end 98.425 53.1) (width 0.25) (layer "F.Cu") (net 23))
+  (segment (start 96.9 76.8) (end 106.15 76.8) (width 0.25) (layer "F.Cu") (net 23))
+  (segment (start 93.5 75.7) (end 93.5 73.525) (width 0.25) (layer "F.Cu") (net 23))
   (segment (start 114 79) (end 114 104.49) (width 0.25) (layer "F.Cu") (net 23))
+  (segment (start 111 82.7) (end 105.8 77.5) (width 0.25) (layer "F.Cu") (net 23))
   (segment (start 96 73.525) (end 96 55.525) (width 0.25) (layer "F.Cu") (net 23))
+  (segment (start 94.8 56.825) (end 94.8 74.7) (width 0.25) (layer "F.Cu") (net 23))
+  (segment (start 95.3 77.5) (end 93.5 75.7) (width 0.25) (layer "F.Cu") (net 23))
+  (segment (start 112 82.65) (end 112 116.7) (width 0.25) (layer "F.Cu") (net 23))
+  (segment (start 117.15 124.35) (end 111 118.2) (width 0.25) (layer "F.Cu") (net 23))
   (segment (start 113 54.475) (end 113 72.475) (width 0.254) (layer "F.Cu") (net 23))
+  (segment (start 106.15 76.8) (end 112 82.65) (width 0.25) (layer "F.Cu") (net 23))
   (segment (start 111.625 53.1) (end 113 54.475) (width 0.25) (layer "F.Cu") (net 23))
   (segment (start 114 104.49) (end 118.62 109.11) (width 0.25) (layer "F.Cu") (net 23))
+  (segment (start 112 116.7) (end 117.11 121.81) (width 0.25) (layer "F.Cu") (net 23))
   (segment (start 126.25 133.5) (end 126.25 137.6625) (width 0.254) (layer "F.Cu") (net 24))
   (segment (start 118.62 131.97) (end 122.18 131.97) (width 0.254) (layer "F.Cu") (net 25))
@@
   (segment (start 118.62 101.49) (end 116 98.87) (width 0.254) (layer "F.Cu") (net 33))
   (segment (start 116 98.87) (end 116 75.5) (width 0.254) (layer "F.Cu") (net 33))
-  (segment (start 93.5 64.525) (end 92.2 65.825) (width 0.25) (layer "F.Cu") (net 35))
-  (segment (start 110 119.7) (end 117.19 126.89) (width 0.25) (layer "F.Cu") (net 35))
-  (segment (start 94.5 78.2) (end 105.4 78.2) (width 0.25) (layer "F.Cu") (net 35))
-  (segment (start 105.4 78.2) (end 110 82.8) (width 0.25) (layer "F.Cu") (net 35))
-  (segment (start 92.2 65.825) (end 92.2 75.9) (width 0.25) (layer "F.Cu") (net 35))
-  (segment (start 92.2 75.9) (end 94.5 78.2) (width 0.25) (layer "F.Cu") (net 35))
-  (segment (start 110 82.8) (end 110 119.7) (width 0.25) (layer "F.Cu") (net 35))
-  (segment (start 117.19 126.89) (end 118.62 126.89) (width 0.25) (layer "F.Cu") (net 35))
-  (segment (start 105.8 77.5) (end 95.3 77.5) (width 0.25) (layer "F.Cu") (net 36))
-  (segment (start 111 118.2) (end 111 82.7) (width 0.25) (layer "F.Cu") (net 36))
-  (segment (start 94.8 74.7) (end 96.9 76.8) (width 0.25) (layer "F.Cu") (net 36))
-  (segment (start 117.11 121.81) (end 118.62 121.81) (width 0.25) (layer "F.Cu") (net 36))
-  (segment (start 93.5 55.525) (end 94.8 56.825) (width 0.25) (layer "F.Cu") (net 36))
-  (segment (start 118.62 124.35) (end 117.15 124.35) (width 0.25) (layer "F.Cu") (net 36))
-  (segment (start 96.9 76.8) (end 106.15 76.8) (width 0.25) (layer "F.Cu") (net 36))
-  (segment (start 93.5 75.7) (end 93.5 73.525) (width 0.25) (layer "F.Cu") (net 36))
-  (segment (start 111 82.7) (end 105.8 77.5) (width 0.25) (layer "F.Cu") (net 36))
-  (segment (start 94.8 56.825) (end 94.8 74.7) (width 0.25) (layer "F.Cu") (net 36))
-  (segment (start 95.3 77.5) (end 93.5 75.7) (width 0.25) (layer "F.Cu") (net 36))
-  (segment (start 112 82.65) (end 112 116.7) (width 0.25) (layer "F.Cu") (net 36))
-  (segment (start 117.15 124.35) (end 111 118.2) (width 0.25) (layer "F.Cu") (net 36))
-  (segment (start 106.15 76.8) (end 112 82.65) (width 0.25) (layer "F.Cu") (net 36))
-  (segment (start 112 116.7) (end 117.11 121.81) (width 0.25) (layer "F.Cu") (net 36))
   (zone locked (net 2) (net_name "GND") (layers F&B.Cu) (hatch edge 0.508)
     (connect_pads thru_hole_only (clearance 0.254))
