File: pcb/main_pcb/main_pcb.kicad_pcb (KiCad board)
At the start: 2 copper layers, 80 x 100 mm, 25 parts, among them J1 Conn_01x05, J10 Conn_01x06_Male, J2 Conn_01x05, J3 Conn_01x05, J4 Conn_01x05, J5 Conn_01x05, J6 Conn_01x05, J7 Conn_01x05, J8 Conn_01x06_Male, U3 DRV8833

Commit message: changes
Routing:
- net /microcontroller/SCL2: track 244.8 -> 93.5 mm
- net /microcontroller/LCS6: track 0.00 -> 151.2 mm
- net /microcontroller/LCS5: track 0.00 -> 81.1 mm
- net /microcontroller/SDA2: track 184.9 -> 103.9 mm
Changed lines of the file:
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@@
   (segment (start 110.5 72.475) (end 110.5 59.4) (width 0.254) (layer "F.Cu") (net 22))
   (segment (start 110.5 77.5) (end 110.5 72.475) (width 0.254) (layer "F.Cu") (net 22))
-  (segment (start 93.5 64.525) (end 92.2 65.825) (width 0.25) (layer "F.Cu") (net 22))
   (segment (start 115.8875 59.5) (end 113.8 59.5) (width 0.254) (layer "F.Cu") (net 22))
-  (segment (start 110 119.7) (end 117.19 126.89) (width 0.25) (layer "F.Cu") (net 22))
   (segment (start 121 110) (end 120.5 110.5) (width 0.254) (layer "F.Cu") (net 22))
-  (segment (start 94.5 78.2) (end 105.4 78.2) (width 0.25) (layer "F.Cu") (net 22))
   (segment (start 113 106.35) (end 113 80) (width 0.254) (layer "F.Cu") (net 22))
   (segment (start 118.62 106.57) (end 120.57 106.57) (width 0.254) (layer "F.Cu") (net 22))
   (segment (start 98.5 57.5) (end 110.4 57.5) (width 0.25) (layer "F.Cu") (net 22))
-  (segment (start 105.4 78.2) (end 110 82.8) (width 0.25) (layer "F.Cu") (net 22))
   (segment (start 98.5 57.5) (end 98.5 73.525) (width 0.25) (layer "F.Cu") (net 22))
   (segment (start 117.15 110.5) (end 113 106.35) (width 0.254) (layer "F.Cu") (net 22))
@@
   (segment (start 110.5 57.4) (end 110.5 54.475) (width 0.254) (layer "F.Cu") (net 22))
   (segment (start 120.57 106.57) (end 121 107) (width 0.254) (layer "F.Cu") (net 22))
-  (segment (start 92.2 65.825) (end 92.2 75.9) (width 0.25) (layer "F.Cu") (net 22))
   (segment (start 121 107) (end 121 110) (width 0.254) (layer "F.Cu") (net 22))
   (segment (start 110.5 59.4) (end 110.5 57.4) (width 0.254) (layer "F.Cu") (net 22))
-  (segment (start 92.2 75.9) (end 94.5 78.2) (width 0.25) (layer "F.Cu") (net 22))
-  (segment (start 110 82.8) (end 110 119.7) (width 0.25) (layer "F.Cu") (net 22))
-  (segment (start 117.19 126.89) (end 118.62 126.89) (width 0.25) (layer "F.Cu") (net 22))
   (segment (start 113 80) (end 110.5 77.5) (width 0.254) (layer "F.Cu") (net 22))
   (via (at 112.2 59.5) (size 0.8) (drill 0.4) (layers "F.Cu" "B.Cu") (net 22))
@@
   (segment (start 113.8 59.5) (end 112.2 59.5) (width 0.254) (layer "B.Cu") (net 22))
   (segment (start 113 72.475) (end 113 78) (width 0.25) (layer "F.Cu") (net 23))
-  (segment (start 105.8 77.5) (end 95.3 77.5) (width 0.25) (layer "F.Cu") (net 23))
-  (segment (start 111 118.2) (end 111 82.7) (width 0.25) (layer "F.Cu") (net 23))
-  (segment (start 94.8 74.7) (end 96.9 76.8) (width 0.25) (layer "F.Cu") (net 23))
-  (segment (start 117.11 121.81) (end 118.62 121.81) (width 0.25) (layer "F.Cu") (net 23))
   (segment (start 113 78) (end 114 79) (width 0.25) (layer "F.Cu") (net 23))
   (segment (start 98.425 53.1) (end 111.625 53.1) (width 0.25) (layer "F.Cu") (net 23))
-  (segment (start 93.5 55.525) (end 94.8 56.825) (width 0.25) (layer "F.Cu") (net 23))
-  (segment (start 118.62 124.35) (end 117.15 124.35) (width 0.25) (layer "F.Cu") (net 23))
   (segment (start 96 55.525) (end 98.425 53.1) (width 0.25) (layer "F.Cu") (net 23))
-  (segment (start 96.9 76.8) (end 106.15 76.8) (width 0.25) (layer "F.Cu") (net 23))
-  (segment (start 93.5 75.7) (end 93.5 73.525) (width 0.25) (layer "F.Cu") (net 23))
   (segment (start 114 79) (end 114 104.49) (width 0.25) (layer "F.Cu") (net 23))
-  (segment (start 111 82.7) (end 105.8 77.5) (width 0.25) (layer "F.Cu") (net 23))
   (segment (start 96 73.525) (end 96 55.525) (width 0.25) (layer "F.Cu") (net 23))
-  (segment (start 94.8 56.825) (end 94.8 74.7) (width 0.25) (layer "F.Cu") (net 23))
-  (segment (start 95.3 77.5) (end 93.5 75.7) (width 0.25) (layer "F.Cu") (net 23))
-  (segment (start 112 82.65) (end 112 116.7) (width 0.25) (layer "F.Cu") (net 23))
-  (segment (start 117.15 124.35) (end 111 118.2) (width 0.25) (layer "F.Cu") (net 23))
   (segment (start 113 54.475) (end 113 72.475) (width 0.254) (layer "F.Cu") (net 23))
-  (segment (start 106.15 76.8) (end 112 82.65) (width 0.25) (layer "F.Cu") (net 23))
   (segment (start 111.625 53.1) (end 113 54.475) (width 0.25) (layer "F.Cu") (net 23))
   (segment (start 114 104.49) (end 118.62 109.11) (width 0.25) (layer "F.Cu") (net 23))
-  (segment (start 112 116.7) (end 117.11 121.81) (width 0.25) (layer "F.Cu") (net 23))
   (segment (start 126.25 133.5) (end 126.25 137.6625) (width 0.254) (layer "F.Cu") (net 24))
   (segment (start 118.62 131.97) (end 122.18 131.97) (width 0.254) (layer "F.Cu") (net 25))
@@
   (segment (start 118.62 101.49) (end 116 98.87) (width 0.254) (layer "F.Cu") (net 33))
   (segment (start 116 98.87) (end 116 75.5) (width 0.254) (layer "F.Cu") (net 33))
+  (segment (start 93.5 64.525) (end 92.2 65.825) (width 0.25) (layer "F.Cu") (net 35))
+  (segment (start 110 119.7) (end 117.19 126.89) (width 0.25) (layer "F.Cu") (net 35))
+  (segment (start 94.5 78.2) (end 105.4 78.2) (width 0.25) (layer "F.Cu") (net 35))
+  (segment (start 105.4 78.2) (end 110 82.8) (width 0.25) (layer "F.Cu") (net 35))
+  (segment (start 92.2 65.825) (end 92.2 75.9) (width 0.25) (layer "F.Cu") (net 35))
+  (segment (start 92.2 75.9) (end 94.5 78.2) (width 0.25) (layer "F.Cu") (net 35))
+  (segment (start 110 82.8) (end 110 119.7) (width 0.25) (layer "F.Cu") (net 35))
+  (segment (start 117.19 126.89) (end 118.62 126.89) (width 0.25) (layer "F.Cu") (net 35))
+  (segment (start 105.8 77.5) (end 95.3 77.5) (width 0.25) (layer "F.Cu") (net 36))
+  (segment (start 111 118.2) (end 111 82.7) (width 0.25) (layer "F.Cu") (net 36))
+  (segment (start 94.8 74.7) (end 96.9 76.8) (width 0.25) (layer "F.Cu") (net 36))
+  (segment (start 117.11 121.81) (end 118.62 121.81) (width 0.25) (layer "F.Cu") (net 36))
+  (segment (start 93.5 55.525) (end 94.8 56.825) (width 0.25) (layer "F.Cu") (net 36))
+  (segment (start 118.62 124.35) (end 117.15 124.35) (width 0.25) (layer "F.Cu") (net 36))
+  (segment (start 96.9 76.8) (end 106.15 76.8) (width 0.25) (layer "F.Cu") (net 36))
+  (segment (start 93.5 75.7) (end 93.5 73.525) (width 0.25) (layer "F.Cu") (net 36))
+  (segment (start 111 82.7) (end 105.8 77.5) (width 0.25) (layer "F.Cu") (net 36))
+  (segment (start 94.8 56.825) (end 94.8 74.7) (width 0.25) (layer "F.Cu") (net 36))
+  (segment (start 95.3 77.5) (end 93.5 75.7) (width 0.25) (layer "F.Cu") (net 36))
+  (segment (start 112 82.65) (end 112 116.7) (width 0.25) (layer "F.Cu") (net 36))
+  (segment (start 117.15 124.35) (end 111 118.2) (width 0.25) (layer "F.Cu") (net 36))
+  (segment (start 106.15 76.8) (end 112 82.65) (width 0.25) (layer "F.Cu") (net 36))
+  (segment (start 112 116.7) (end 117.11 121.81) (width 0.25) (layer "F.Cu") (net 36))
   (zone locked (net 2) (net_name "GND") (layers F&B.Cu) (hatch edge 0.508)
     (connect_pads thru_hole_only (clearance 0.254))
