File: pcb/main_pcb/microcontroller.kicad_sch (KiCad schematic)
At the start: 20 parts, among them J1 Conn_01x05, J10 Conn_01x06_Male, J2 Conn_01x05, J3 Conn_01x05, J4 Conn_01x05, J5 Conn_01x05, J6 Conn_01x05, J7 Conn_01x05, J8 Conn_01x06_Male, U2 Teensy_4.0, U3 DRV8833

Commit message: changes to PCB
Parts:
- added U?: Teensy_4.0, symbol sym_library:Teensy_4.0
- added U?: Teensy_4.0, symbol sym_library:Teensy_4.1
- U2: symbol sym_library:Teensy_4.1 -> sym_library:Teensy_4.0
Connections:
- net +BATT: now also U?.48 (VIN); no longer U2.48 (VIN)
- net AEQ1: now also U?.13 (IO11); no longer U2.13 (IO11)
- net AEQ2: now also U?.14 (IO12); no longer U2.14 (IO12)
- net AIN1: now also U?.4 (IO2); no longer U2.4 (IO2)
- net AIN2: now also U?.11 (IO9); no longer U2.11 (IO9)
- net BEQ1: now also U?.2 (IO0); no longer U2.2 (IO0)
- net BEQ2: now also U?.3 (IO1); no longer U2.3 (IO1)
- net BIN1: now also U?.10 (IO8); no longer U2.10 (IO8)
- net BIN2: now also U?.5 (IO3); no longer U2.5 (IO3)
- net GND: now also U?. (VBat); no longer U2. (VBat)
- net LCS1: now also U?.20 (IO18); no longer U2.20 (IO18)
- net LCS2: now also U?. (VBat)
- net LCS3: now also U?.16 (IO22)
- net LCS4: now also U?.8 (IO6); no longer U2.8 (IO6)
- net LCS5: now also U?.22 (IO16); no longer U2.22 (IO16)
- net LCS6: now also U?.23 (IO15); no longer U2.23 (IO15)
- net LCS7: now also U?.24 (IO14); no longer U2.24 (IO14)
- net LED0: now also U?.6 (IO4); no longer U2.6 (IO4)
- net LED1: now also U?.7 (IO5); no longer U2.7 (IO5)
- net LED2: now also U?.18 (IO20); no longer U2.18 (IO20)
- net LED3: now also U?.19 (IO19); no longer U2.19 (IO19)
- net SCL2: now also U?.21 (IO17); no longer U2.21 (IO17)
- no-connect marks 14 -> 23

Commit message: changes
Parts:
- removed U2, U?: Teensy_4.0, symbol sym_library:Teensy_4.0
- gave numbers to parts that had none: 1
Connections:
- no-connect marks 23 -> 14
